File: HGHardware.sch (KiCad schematic (older format))
At the start: 108 parts, among them J1 Conn_01x04_Male, J2 SWD Conn, J3 USB_C_Receptacle_USB2.0, Q1 MMBTA42, Q2 FDS2672CT, SW1 SW_Push, SW2 SW_SPST, SW3 SW_Push, U2 HV507PG-G-MyKiCadLib, U3 ESP-12S, U4 W25Q32FWSSIG, U5 UCC3803, U7 TXS0104EPWR, U9 AOZ1031, Y1 8MHz, Y2 8MHz

Commit message: 原理图修改，同步
Parts:
- removed C18: 100nF, Capacitor_SMD:C_0603_1608Metric, symbol Device:C
- removed U3: ESP-12S, ESP-12S:ESP-12S, symbol ESP-12S:ESP-12S
- removed U4: W25Q32FWSSIG, SOIC127P790X216-8N:SOIC127P790X216-8N, symbol W25Q32FWSSIG:W25Q32FWSSIG
- added D? (x2): LED, symbol Device:LED
- added Q? (x3): S8050, Package_TO_SOT_THT:TO-92_Inline, symbol Transistor_BJT:S8050
- added R? (x5): R, symbol Device:R
- added U?: ESP32-WROOM-32, RF_Module:ESP32-WROOM-32, symbol RF_Module:ESP32-WROOM-32
- added U?: CH340C, Package_SO:SOIC-16_3.9x9.9mm_P1.27mm, symbol Interface_USB:CH340C
- added X?: YSO120TK C669097, symbol Oscillator:SG-3030CM
- J3: symbol HGHardware-rescue:USB_C_Receptacle_USB2.0-Connector -> Connector:USB_C_Receptacle_USB2.0
Connections:
- wire segments 411 -> 406
- no-connect marks 20 -> 18
Other:
- note removed: "ESP-12S has pull-up/down resistor inside."
- moved on the sheet: C10, C11, C12, C13, C14, C15, C16, C21, C22, C23, C26, C27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

Commit message: 20210306完善原理图，升压模块将单独使用
Parts:
- removed C19: 20pF, Capacitor_SMD:C_0603_1608Metric, symbol Device:C
- removed C21: 47uF 16v, Capacitor_SMD:C_1210_3225Metric, symbol HGHardware-rescue:C-NixieSupply5vto170vDCMBoostMini-rescue
- removed C22, C30: 100uF 16v, Capacitor_SMD:C_1210_3225Metric, symbol HGHardware-rescue:C-NixieSupply5vto170vDCMBoostMini-rescue
- removed C23: 10uF, Capacitor_Tantalum_SMD:CP_EIA-3216-18_Kemet-A, symbol Device:C
- removed C25, C35: 100nF, Capacitor_SMD:C_0603_1608Metric, symbol Device:C
- removed C26: 0.1uF, Capacitor_SMD:C_0805_2012Metric, symbol HGHardware-rescue:C-NixieSupply5vto170vDCMBoostMini-rescue
- removed C27: 220pF, Capacitor_SMD:C_0805_2012Metric, symbol HGHardware-rescue:C-NixieSupply5vto170vDCMBoostMini-rescue
- removed C28: 430pF, Capacitor_SMD:C_0805_2012Metric, symbol HGHardware-rescue:C-NixieSupply5vto170vDCMBoostMini-rescue
- removed C29: 0.1uF 16v, Capacitor_SMD:C_0805_2012Metric, symbol HGHardware-rescue:C-NixieSupply5vto170vDCMBoostMini-rescue
- removed C31: 1nF, Capacitor_SMD:C_0805_2012Metric, symbol HGHardware-rescue:C-NixieSupply5vto170vDCMBoostMini-rescue
- removed C32: 560pF 250v, Capacitor_SMD:C_0603_1608Metric, symbol HGHardware-rescue:C-NixieSupply5vto170vDCMBoostMini-rescue
- removed C33: 100pF 250v, Capacitor_SMD:C_0805_2012Metric, symbol HGHardware-rescue:C-NixieSupply5vto170vDCMBoostMini-rescue
- removed C34, C36: 1uF 250v, Capacitor_SMD:C_1812_4532Metric, symbol HGHardware-rescue:C-NixieSupply5vto170vDCMBoostMini-rescue
- removed C37, C38: 0.1uF 250v, Capacitor_SMD:C_0805_2012Metric, symbol HGHardware-rescue:C-NixieSupply5vto170vDCMBoostMini-rescue
- removed C4, C5: C, Capacitor_SMD:C_0603_1608Metric, symbol Device:C
- removed D11: BAT54, Diode_SMD:D_SOD-323_HandSoldering, symbol HGHardware-rescue:D_Schottky-NixieSupply5vto170vDCMBoostMini-rescue
- removed D12: ES1D, Diode_SMD:D_SMA, symbol HGHardware-rescue:D-NixieSupply5vto170vDCMBoostMini-rescue
- removed J1: Conn_01x04_Male, Connector_PinHeader_2.54mm:PinHeader_1x04_P2.54mm_Vertical, symbol Connector:Conn_01x04_Male
- removed J2: SWD Conn, Connector_PinHeader_2.54mm:PinHeader_1x04_P2.54mm_Vertical, symbol Connector:Conn_01x04_Female
- removed L1, L4: 60ohm 100Mhz, Resistor_SMD:R_0805_2012Metric, symbol HGHardware-rescue:L-NixieSupply5vto170vDCMBoostMini-rescue
- removed L2: 33uH, Inductor_SMD:L_12x12mm_H4.5mm, symbol HGHardware-rescue:L-NixieSupply5vto170vDCMBoostMini-rescue
- removed L3: 4.7uH, Inductor_SMD:L_7.3x7.3_H3.5, symbol Device:L
- removed Q1: MMBTA42, Package_TO_SOT_SMD:SOT-23, symbol HGHardware-rescue:MMBT3904-NixieSupply5vto170vDCMBoostMini-rescue
- removed Q2: FDS2672CT, Package_SO:SO-8_3.9x4.9mm_P1.27mm, symbol HGHardware-rescue:FDMS86255ET150-NixieSupply5vto170vDCMBoostMini-rescue
- removed Q?: S8050, Package_TO_SOT_THT:TO-92_Inline, symbol Transistor_BJT:S8050
- removed R10, R25: 1k, Resistor_SMD:R_0805_2012Metric, symbol HGHardware-rescue:R-NixieSupply5vto170vDCMBoostMini-rescue
- removed R11, R34: 10KO, Resistor_SMD:R_0603_1608Metric, symbol Device:R
- removed R14, R20: 100k, Resistor_SMD:R_0805_2012Metric, symbol HGHardware-rescue:R-NixieSupply5vto170vDCMBoostMini-rescue
- removed R15: 2k, Resistor_SMD:R_0805_2012Metric, symbol HGHardware-rescue:R-NixieSupply5vto170vDCMBoostMini-rescue
- removed R21: 60.4k, Resistor_SMD:R_0805_2012Metric, symbol HGHardware-rescue:R-NixieSupply5vto170vDCMBoostMini-rescue
- removed R22: N.U., Resistor_SMD:R_0805_2012Metric, symbol HGHardware-rescue:R-NixieSupply5vto170vDCMBoostMini-rescue
- removed R23: 0 Ohm, Resistor_SMD:R_0805_2012Metric, symbol HGHardware-rescue:R-NixieSupply5vto170vDCMBoostMini-rescue
- removed R24: 4.12k, Resistor_SMD:R_0805_2012Metric, symbol HGHardware-rescue:R-NixieSupply5vto170vDCMBoostMini-rescue
- removed R26: 0.1 1/2W, Resistor_SMD:R_0805_2012Metric, symbol HGHardware-rescue:R-NixieSupply5vto170vDCMBoostMini-rescue
- removed R27: 634k, Resistor_SMD:R_0805_2012Metric, symbol HGHardware-rescue:R-NixieSupply5vto170vDCMBoostMini-rescue
- removed R28: 7.68k, Resistor_SMD:R_0805_2012Metric, symbol HGHardware-rescue:R-NixieSupply5vto170vDCMBoostMini-rescue
- removed R33: 1KO, Resistor_SMD:R_0603_1608Metric, symbol Device:R
- removed R35: 1.5KO, Resistor_SMD:R_0603_1608Metric, symbol Device:R
- removed R?: R, symbol Device:R
- removed SW1, SW3: SW_Push, HGHardware:MyButton, symbol Switch:SW_Push
- removed U5: UCC3803, Package_SO:SO-8_3.9x4.9mm_P1.27mm, symbol HGHardware-rescue:AAC243-NixieSupply5vto170vDCMBoostMini-rescue
- removed U9: AOZ1031, Package_SO:SOIC-8_3.9x4.9mm_P1.27mm, symbol HGHardware-rescue:AOZ1031
- removed Y1, Y2: 8MHz, Crystal:Crystal_SMD_5032-2Pin_5.0x3.2mm, symbol Device:Crystal
- added C18: 22uF, Capacitor_SMD:C_0603_1608Metric, symbol Device:C
- added C?: 10uF, Capacitor_SMD:C_0603_1608Metric, symbol Device:C
- added C?: 100nF, Capacitor_SMD:C_0603_1608Metric, symbol Device:C
- added D11, D12: RED, LED_SMD:LED_0603_1608Metric, symbol Device:LED
- added J?: Micro_SD_Card, symbol Connector:Micro_SD_Card
- added J?: JTAG, symbol Connector_Generic_Shielded:Conn_01x06_Shielded
- added L2: 2.2uH, Inductor_SMD:L_0805_2012Metric, symbol Device:L
- added Q?: S8050, symbol Transistor_BJT:S8050
- added R14, R15: 1KΩ, Resistor_SMD:R_0603_1608Metric, symbol Device:R
- added R23: 100KΩ, Resistor_SMD:R_0603_1608Metric, symbol Device:R
- added R24: 30KΩ, Resistor_SMD:R_0603_1608Metric, symbol Device:R
- added R25, R?: 10KΩ, Resistor_SMD:R_0603_1608Metric, symbol Device:R
- added R26: 0Ω, Resistor_SMD:R_0603_1608Metric, symbol Device:R
- added R8: 120Ω, Resistor_SMD:R_0603_1608Metric, symbol Device:R
- added U5: TPS563201DDCR, Package_TO_SOT_SMD:SOT-23-6, symbol Regulator_Switching:TPS563200
- C1: value 100nF -> 10uF
- C15: value 10uF -> 100uF
- C17, C7: value 20pF -> 100nF
- C2: value C -> 100nF
- C6: value 20pF -> 22uF
- D1: value WS2812B-2020 -> WS2812B×6
- D10: renamed from D?; value LED -> BLUE; footprint (none) -> LED_SMD:LED_0603_1608Metric
- D13: value LED -> RED
- D9: renamed from D?; value LED -> GREEN; footprint (none) -> LED_SMD:LED_0603_1608Metric
- J3: footprint HGHardware:USB TypeC 6P Horizontal -> Connector_USB:USB_C_Receptacle_HRO_TYPE-C-31-M-12
- N6: value NixieTube -> NixieTube×6
- Q1, Q3: renamed from Q?; footprint Package_TO_SOT_THT:TO-92_Inline -> (none)
- R1, R2, R3, R4, R5, R6: value 33KO -> 33KΩ
- R10, R9: renamed from R?; value R -> 10KΩ; footprint (none) -> Resistor_SMD:R_0603_1608Metric
- R11, R12: renamed from R?; value R -> 1KΩ; footprint (none) -> Resistor_SMD:R_0603_1608Metric
- R13: value 31.1KO -> 1KΩ
- R17: value 510KO -> 510KΩ
- R29, R30: value 5.1K -> 5.1KΩ
- R7: value 10KO -> 120Ω
- SW2: footprint Button_Switch_THT:SW_DIP_SPSTx01_Slide_6.7x4.1mm_W7.62mm_P2.54mm_LowProfile -> (none)
- U2: value HV507PG-G-MyKiCadLib -> HV507PG-G; footprint QFP80P2390X1790X340-80N:QFP80P2390X1790X340-80N -> HGHardware:QFP80P2390X1790X340-80N; symbol HGHardware-rescue:HV507PG-G-MyKiCadLib -> MyLib:HV507PG-G
- gave numbers to parts that had none: 3
Connections:
- net labels added: CH340_DTR, CH340_RTS, CH340_RXD, CH340_TXD, ESP32_EN, ESP32_IO0, ESP32_IO12, ESP32_IO13, ESP32_IO14, ESP32_IO15, ESP32_IO16, ESP32_IO17, ESP32_IO18, ESP32_IO19, ESP32_IO2, ESP32_IO21, ESP32_IO22, ESP32_IO23, ESP32_IO25, ESP32_IO26, ESP32_IO27, ESP32_IO32, ESP32_IO33, ESP32_IO34, ESP32_IO35, ESP32_IO4, ESP32_IO5, ESP32_RXD0, ESP32_TXD0, SD_CLK, SD_CMD, SD_DAT0, SD_DAT1, SD_DAT2, SD_DAT3, USB_D+, USB_D-
- net labels removed: BOOT0, DAC_OUT1, GNDPWR, NRST, QSPI_CS, QSPI_IO0, QSPI_IO1, QSPI_IO2, QSPI_IO3, QSPI_SCK, SWCLK, SWDIO, UART1_RX, UART1_TX, VPP_EN, WKP1
- wire segments 406 -> 320
- no-connect marks 18 -> 17
Other:
- note added: "The following pins can only be used as input pins: SENSOR_VP SENSOR_VN IO34 IO35."
- note removed: "OUTPUT SET to 167Volts"
- moved on the sheet: C14, C15, C16, C20, C24, D10, D7, D8, D9, H1, H2, H3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

Commit message: 犹豫不决ing
Parts:
- removed C?: 10uF, Capacitor_SMD:C_0603_1608Metric, symbol Device:C
- removed C?: 100nF, Capacitor_SMD:C_0603_1608Metric, symbol Device:C
- removed J?: Micro_SD_Card, symbol Connector:Micro_SD_Card
- removed J?: JTAG, symbol Connector_Generic_Shielded:Conn_01x06_Shielded
- removed Q1, Q3, Q?: S8050, symbol Transistor_BJT:S8050
- removed R26: 0Ω, Resistor_SMD:R_0603_1608Metric, symbol Device:R
- removed SW2: SW_SPST, symbol Switch:SW_SPST
- removed U1: CH340C, Package_SO:SOIC-16_3.9x9.9mm_P1.27mm, symbol Interface_USB:CH340C
- removed X1: YSO120TK C669097, symbol Oscillator:SG-3030CM
- added C7, C8: C, Capacitor_SMD:C_0603_1608Metric, symbol Device:C
- added J3: Conn_01x06, Connector_PinHeader_2.54mm:PinHeader_1x06_P2.54mm_Vertical, symbol Connector_Generic:Conn_01x06
- added Q1, Q2, Q3: S8050, Package_TO_SOT_SMD:SOT-23, symbol Device:Q_NPN_BEC
- added R4: NC, Resistor_SMD:R_0603_1608Metric, symbol Device:R
- added U2: ES8388, Package_DFN_QFN:QFN-28-1EP_4x4mm_P0.4mm_EP2.4x2.4mm_ThermalVias, symbol MyLib:ES8388
- added U3: CH340K, Package_SO:SSOP-10_3.9x4.9mm_P1.00mm, symbol MyLib:CH340K
- added Y1: 32.738kHz, Crystal:Crystal_SMD_2012-2Pin_2.0x1.2mm, symbol Device:Crystal
- L1: renamed from L2; footprint Inductor_SMD:L_0805_2012Metric -> Inductor_SMD:L_Taiyo-Yuden_MD-4040
- gave numbers to parts that had none: 1
- renumbered C15 to C1, C18 to C10, C20 to C11, C24 to C12, C8 to C15, C9 to C16, C10 to C17, C11 to C18, C12 to C19, C16 to C2, C13 to C20, C14 to C21, C6 to C3, C7 to C4, C1 to C5, C2 to C6, C17 to C9, D13 to D10, D5 to D11, D8 to D12, D6 to D13, D7 to D5, D9 to D6, D10 to D7, D11 to D8, D12 to D9, J3 to J1, R29 to R1, R9 to R11, R10 to R12, R2 to R14, R11 to R15, R12 to R16, R13 to R17, R14 to R18, R15 to R19, R30 to R2, R17 to R20, R16 to R21, R3 to R22, R18 to R23, R19 to R24, R4 to R25, R5 to R26, R6 to R27, R23 to R3, R7 to R5, R8 to R6, R24 to R7, R25 to R8, R1 to R9, U3 to U1, U5 to U4, U7 to U5, U2 to U6
Connections:
- net +3V3: now also C10.2, L1.2, R7.1, J3.1 (Pin_1), U3.10 (V3), U3.7 (VCC)
- net +5V: now also J1.A4 (VBUS), J1.A9 (VBUS), J1.B4 (VBUS), J1.B9 (VBUS)
- net CH340_DTR: now also Q2.3 (C), Q3.3 (C), U3.4 (~DTR)
- net CH340_RTS: now also Q1.2 (E), U3.6 (~RTS)
- net ESP32_EN: now also Q1.3 (C)
- net ESP32_IO0: now also Q2.2 (E)
- net ESP32_IO12: now also J3.4 (Pin_4)
- net ESP32_IO13: now also J3.5 (Pin_5)
- net ESP32_IO14: now also J3.6 (Pin_6)
- net ESP32_IO15: now also J3.3 (Pin_3)
- net ESP32_IO2: now also Q3.2 (E)
- net GNDD: now also C7.1, C8.1, J3.2 (Pin_2), U3.3 (GND)
- net USB_D+: now also U3.1 (UD+)
- net USB_D-: now also U3.2 (UD-)
- net at R13.1: now also Q3.1 (B)
- net at R5.2: now also U3.8 (TXD)
- net at R6.2: now also U3.9 (RXD)
- net at R11.1: now also Q1.1 (B)
- net at R12.1: now also Q2.1 (B)
- net ESP32_IO32 renamed 32K_XP
- net 32K_XP: now also C7.2, R4.1, Y1.1
- net ESP32_IO33 renamed 32K_XN
- net 32K_XN: now also C8.2, R4.2, Y1.2
- no-connect marks 17 -> 13
Other:
- note added: "Be careful! Kicad's 8050 and SOT-23 footprint are not same pins order."
- note added: "JTAG and SD card are only valid one time."
- moved on the sheet: C5, C6, R11, R12, R13, R5, R6
