File: Audio.sch (KiCad schematic (older format))
At the start: 0 parts

Commit message: 同步
Parts:
- added C? (x10): C, symbol Device:C
- added MK?: Microphone, symbol Device:Microphone
- added R?: 0, symbol Device:R
- added R?: 10K, symbol Device:R
- added U?: ES8311, symbol MyLib:ES8311
Connections:
- new net: C?.2, U?.14 (DACVREF)
- new net: C?.2, U?.16 (VMID)
- new net: R?.1, U?.20 (CE)
- new net +3.3VA: C?.1, C?.1, C?.1, R?.1, U?.11 (AVDD), U?.3 (PVDD), U?.4 (DVDD)
- new net +3V3: R?.2
- new net ADCVREF: C?.2, U?.15 (ADCVREF)
- new net Codec_I2C_SCL: U?.1 (CCLK)
- new net Codec_I2C_SDA: U?.19 (CDATA)
- new net Codec_I2S_LRCK: U?.8 (LRCK)
- new net Codec_I2S_MCLK: U?.2 (MCLK)
- new net Codec_I2S_SCLK: U?.6 (SCLK)
- new net Codec_I2S_SDI: U?.9 (DSDIN)
- new net Codec_I2S_SDO: U?.7 (ASDOUT)
- new net GNDA: C?.1, C?.1, C?.1, C?.2, C?.2, C?.2, U?.10 (AGND), U?.21 (PGND)
- new net GNDD: R?.2, U?.5 (DGND)
