File: NixieTubeBoard/NixieTubeBoard.kicad_pcb (KiCad board)
At the start: 2 copper layers, 100 x 50 mm, 26 parts, among them U6 HV507PG-G

Commit message: 同步
Changed lines of the file:
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@@
-(kicad_pcb (version 20171130) (host pcbnew 5.1.9)
+(kicad_pcb (version 20171130) (host pcbnew "(5.1.8)-1")
   (general
     (thickness 1.6)
@@
   )
   (setup
-    (last_trace_width 0.5)
+    (last_trace_width 0.25)
     (user_trace_width 0.5)
     (trace_clearance 0.125)
@@
     (pad_to_mask_clearance 0)
     (aux_axis_origin 0 0)
-    (visible_elements FFFFFF7F)
+    (visible_elements 7FFFFFFF)
     (pcbplotparams
       (layerselection 0x010fc_ffffffff)
@@
   (segment (start 118.525 82.525) (end 118.5 82.5) (width 0.5) (layer F.Cu) (net 75))
   (segment (start 119.5 82.525) (end 118.525 82.525) (width 0.5) (layer F.Cu) (net 75))
-  (via (at 126.5 83.5) (size 0.6) (drill 0.3) (layers F.Cu B.Cu) (net 75))
-  (segment (start 126.45 83.55) (end 126.5 83.5) (width 0.5) (layer F.Cu) (net 75))
-  (segment (start 126.45 84.6) (end 126.45 83.55) (width 0.5) (layer F.Cu) (net 75))
   (via (at 142.5 83.5) (size 0.6) (drill 0.3) (layers F.Cu B.Cu) (net 75))
   (segment (start 142.45 83.55) (end 142.5 83.5) (width 0.5) (layer F.Cu) (net 75))
@@
   (segment (start 178.525 82.525) (end 178.5 82.5) (width 0.5) (layer F.Cu) (net 75))
   (segment (start 179.5 82.525) (end 178.525 82.525) (width 0.5) (layer F.Cu) (net 75))
+  (via (at 127 84.99999) (size 0.6) (drill 0.3) (layers F.Cu B.Cu) (net 75))
+  (segment (start 126.45 84.6) (end 126.84999 84.99999) (width 0.5) (layer F.Cu) (net 75))
+  (segment (start 126.84999 84.99999) (end 127 84.99999) (width 0.5) (layer F.Cu) (net 75))
   (segment (start 172.214002 82.4) (end 171.45 82.4) (width 0.25) (layer F.Cu) (net 79))
   (segment (start 174.414002 84.6) (end 172.214002 82.4) (width 0.25) (layer F.Cu) (net 79))
