File: NixieTubeBoard/NixieTubeBoard.sch (KiCad schematic (older format))
At the start: 26 parts, among them U6 HV507PG-G

Commit message: 同步
Parts:
- added J?: Conn_01x06, symbol Connector_Generic:Conn_01x06
- added J?: Conn_01x02, symbol Connector_Generic:Conn_01x02
Connections:
- net +5V: now also J?.5 (Pin_5)
- net GND: now also J?.2 (Pin_2), J?.6 (Pin_6)
- net HV_CLK_5V: now also J?.1 (Pin_1)
- net HV_DIN_5V: now also J?.3 (Pin_3)
- net HV_LE_5V: now also J?.2 (Pin_2)
- net ND1: now also U6.24 (HVOUT64)
- net ND2: now also U6.23 (HVOUT63)
- net ND3: now also U6.41 (HVOUT1)
- net ND4: now also U6.42 (HVOUT2)
- net RGBLED_5V: now also J?.4 (Pin_4)
- net VPP: now also J?.1 (Pin_1)
Changed lines of the file:
@@
 	9850 5950 10400 5950
 Wire Wire Line
-	7100 4250 7650 4250
+	9850 2950 10400 2950
 $Comp
 L Device:C C15
@@
 $EndComp
 Wire Wire Line
-	7100 4150 7650 4150
-Wire Wire Line
-	7100 4350 7650 4350
+	9850 2850 10400 2850
+Wire Wire Line
+	7900 2850 8450 2850
 Wire Wire Line
 	9850 4050 10400 4050
@@
 $EndComp
 Wire Wire Line
-	7100 4450 7650 4450
+	7900 2950 8450 2950
 NoConn ~ 7250 5500
-Text Label 7650 4250 2    50   ~ 0
+Text Label 10400 2950 2    50   ~ 0
 ND2
-Text Label 7650 4150 2    50   ~ 0
+Text Label 10400 2850 2    50   ~ 0
 ND1
-Text Label 7100 4450 0    50   ~ 0
+Text Label 7900 2950 0    50   ~ 0
 ND4
-Text Label 7100 4350 0    50   ~ 0
+Text Label 7900 2850 0    50   ~ 0
 ND3
 Wire Wire Line
@@
 Wire Wire Line
 	5500 2850 5600 2850
+$Comp
+L Connector_Generic:Conn_01x06 J?
+U 1 1 604B7938
+P 3200 5200
+F 0 "J?" H 3280 5192 50  0000 L CNN
+F 1 "Conn_01x06" H 3280 5101 50  0000 L CNN
+F 2 "" H 3200 5200 50  0001 C CNN
+F 3 "~" H 3200 5200 50  0001 C CNN
+	1    3200 5200
+	1    0    0    -1
+$EndComp
+Text Label 2550 5000 0    50   ~ 0
+HV_CLK_5V
+Wire Wire Line
+	2550 5000 3000 5000
+Wire Wire Line
+	3000 5100 2550 5100
+Wire Wire Line
+	3000 5200 2550 5200
+Wire Wire Line
+	3000 5300 2550 5300
+Wire Wire Line
+	3000 5400 2550 5400
+Wire Wire Line
+	3000 5500 2550 5500
+Text Label 2550 5100 0    50   ~ 0
+HV_LE_5V
+Text Label 2550 5200 0    50   ~ 0
+HV_DIN_5V
+$Comp
+L power:GNDD #PWR?
+U 1 1 604FC080
+P 2550 5500
+F 0 "#PWR?" H 2550 5250 50  0001 C CNN
+F 1 "GNDD" H 2554 5345 50  0000 C CNN
+F 2 "" H 2550 5500 50  0001 C CNN
+F 3 "" H 2550 5500 50  0001 C CNN
+	1    2550 5500
+	1    0    0    -1
+$EndComp
+$Comp
+L power:+5V #PWR?
+U 1 1 604FCB8A
+P 2550 5400
+F 0 "#PWR?" H 2550 5250 50  0001 C CNN
+F 1 "+5V" H 2450 5500 50  0000 C CNN
+F 2 "" H 2550 5400 50  0001 C CNN
+F 3 "" H 2550 5400 50  0001 C CNN
+	1    2550 5400
+	1    0    0    -1
+$EndComp
+$Comp
+L Connector_Generic:Conn_01x02 J?
+U 1 1 604FCF9D
+P 3200 6000
+F 0 "J?" H 3280 5992 50  0000 L CNN
+F 1 "Conn_01x02" H 3280 5901 50  0000 L CNN
+F 2 "" H 3200 6000 50  0001 C CNN
+F 3 "~" H 3200 6000 50  0001 C CNN
+	1    3200 6000
+	1    0    0    -1
+$EndComp
+$Comp
+L power:GND #PWR?
+U 1 1 604FDB27
+P 3000 6100
+F 0 "#PWR?" H 3000 5850 50  0001 C CNN
+F 1 "GND" V 3005 5972 50  0000 R CNN
+F 2 "" H 3000 6100 50  0001 C CNN
+F 3 "" H 3000 6100 50  0001 C CNN
+	1    3000 6100
+	1    0    0    -1
+$EndComp
+$Comp
+L power:VPP #PWR?
+U 1 1 604FE276
+P 3000 6000
+F 0 "#PWR?" H 3000 5850 50  0001 C CNN
+F 1 "VPP" H 3015 6173 50  0000 C CNN
+F 2 "" H 3000 6000 50  0001 C CNN
+F 3 "" H 3000 6000 50  0001 C CNN
+	1    3000 6000
+	1    0    0    -1
+$EndComp
+Text Label 2550 5300 0    50   ~ 0
+RGBLED_5V
 $EndSCHEMATC
