File: NixieTubeJackBoard/NixieTubeJackBoard.kicad_pcb (KiCad board)
At the start: 2 copper layers, 17.1 x 17.1 mm, 2 parts, among them J1 Conn_01x13_Male, J2 Conn_01x13_Female

Commit message: 拆分得七零八落
Parts:
- turned J1 to 180 degrees
Routing:
- net Net-(J1-Pad4): track 2.31 -> 7.06 mm
- net Net-(J1-Pad11): track 2.31 -> 7.06 mm
- net Net-(J1-Pad2): track 3.27 -> 0.00 mm
- net Net-(J1-Pad13): track 3.27 -> 0.00 mm
- net Net-(J1-Pad3): track 3.85 -> 5.91 mm
- net Net-(J1-Pad12): track 3.85 -> 5.91 mm
- net Net-(J1-Pad5): track 2.75 -> 4.62 mm
- net Net-(J1-Pad10): track 2.75 -> 4.62 mm
- net Net-(J1-Pad9): track 4.27 -> 2.75 mm
- net Net-(J1-Pad6): track 4.27 -> 2.75 mm
- net Net-(J1-Pad1): track 2.00 -> 1.50 mm
Other:
- board size 17.1 x 17.1 mm -> 13.6 x 16.1 mm

Commit message: 改了一堆东西忘了提交了
Routing:
- net Net-(J1-Pad3): track 5.91 -> 6.51 mm
- net Net-(J1-Pad12): track 5.91 -> 6.51 mm
Changed lines of the file:
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@@
-(kicad_pcb (version 20171130) (host pcbnew 5.1.9)
+(kicad_pcb (version 20171130) (host pcbnew "(5.1.8)-1")
   (general
     (thickness 1.6)
@@
     (0 F.Cu signal)
     (31 B.Cu signal)
-    (32 B.Adhes user)
     (33 F.Adhes user)
-    (34 B.Paste user)
     (35 F.Paste user)
-    (36 B.SilkS user)
     (37 F.SilkS user)
     (38 B.Mask user)
@@
     (46 B.CrtYd user)
     (47 F.CrtYd user)
-    (48 B.Fab user)
     (49 F.Fab user)
   )
@@
     (pad_drill 0.762)
     (pad_to_mask_clearance 0)
-    (aux_axis_origin 0 0)
-    (visible_elements FFFFFF7F)
+    (aux_axis_origin 100 100)
+    (visible_elements 7FFFFFFF)
     (pcbplotparams
       (layerselection 0x010fc_ffffffff)
@@
   (gr_line (start 99.5 95.6) (end 100.6 95.6) (layer F.SilkS) (width 0.12))
   (gr_line (start 99.5 95.8) (end 100.6 95.8) (layer F.SilkS) (width 0.12))
-  (segment (start 104.526411 95.546424) (end 104.526411 96.875644) (width 0.5) (layer F.Cu) (net 2))
-  (segment (start 101.979987 93) (end 104.526411 95.546424) (width 0.5) (layer F.Cu) (net 2))
-  (segment (start 101 93) (end 101.979987 93) (width 0.5) (layer F.Cu) (net 2))
+  (segment (start 104.526411 94.526411) (end 104.526411 96.875644) (width 0.5) (layer F.Cu) (net 2))
+  (segment (start 103 93) (end 104.526411 94.526411) (width 0.5) (layer F.Cu) (net 2))
+  (segment (start 101 93) (end 103 93) (width 0.5) (layer F.Cu) (net 2))
   (segment (start 106.19259 104.575267) (end 105.117814 105.650043) (width 0.5) (layer F.Cu) (net 3))
   (segment (start 106.19259 100.069739) (end 106.19259 104.575267) (width 0.5) (layer F.Cu) (net 3))
@@
   (segment (start 93.80741 100.069739) (end 93.80741 104.575267) (width 0.5) (layer F.Cu) (net 10))
   (segment (start 94.540101 99.337048) (end 93.80741 100.069739) (width 0.5) (layer F.Cu) (net 10))
-  (segment (start 98.020013 93) (end 99 93) (width 0.5) (layer F.Cu) (net 11))
-  (segment (start 95.473589 95.546424) (end 98.020013 93) (width 0.5) (layer F.Cu) (net 11))
-  (segment (start 95.473589 96.875644) (end 95.473589 95.546424) (width 0.5) (layer F.Cu) (net 11))
+  (segment (start 97 93) (end 99 93) (width 0.5) (layer F.Cu) (net 11))
+  (segment (start 95.473589 94.526411) (end 97 93) (width 0.5) (layer F.Cu) (net 11))
+  (segment (start 95.473589 96.875644) (end 95.473589 94.526411) (width 0.5) (layer F.Cu) (net 11))
   (segment (start 100 93.000001) (end 100 94.5) (width 0.5) (layer F.Cu) (net 13))
   (zone (net 7) (net_name "Net-(J1-Pad7)") (layer F.Cu) (hatch edge 0.508)
